File: SpectrumAnalyzerCaps.kicad_pcb (KiCad board)
At the start: 2 copper layers, 161.3 x 81.3 mm, 327 parts, among them J1 Conn_01x03_Male, J2 Conn_01x03_Male

Commit message: clean up
Parts:
- moved H2 2.29 mm to (65.3, 151.9)
- moved H4 2.29 mm to (220.6, 152.0)
- moved C63 0.31 mm to (129.5, 90.2)
- moved C151 0.28 mm to (207.6, 76.6)
- moved C32 0.27 mm to (102.7, 82.5)
- moved C43 0.26 mm to (111.8, 90.2)
- moved C33 0.24 mm to (102.9, 90.2)
- moved C23 0.22 mm to (94.0, 90.2)
- moved C102 0.21 mm to (165.1, 82.5)
- moved C13 0.20 mm to (85.1, 90.2)
- moved C150 0.18 mm to (200.7, 143.5)
- moved C20 0.18 mm to (85.1, 143.5)
- moved C30 0.18 mm to (94.0, 143.5)
- moved C140 0.18 mm to (191.8, 143.5)
- moved C156 0.18 mm to (209.6, 113.0)
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Routing:
- net VDD: track 1776.5 -> 1752.5 mm
- net VSS: track 1130.5 -> 1129.3 mm
